File: AlphaStag.kicad_sch (KiCad schematic)
At the start: 89 parts, among them SW1 SW_Push, U1 SRV05-4, U2 ATmega32U4-A, Y1 16MHz

Commit message: routing
Parts:
- removed C3: 4.7uF, Capacitor_SMD:C_0805_2012Metric, symbol device:C_Small
- removed F1: Polyfuse_Small, Fuse:Fuse_1210_3225Metric, symbol device:Polyfuse_Small
- removed U1: SRV05-4, Package_TO_SOT_SMD:SOT-23-6, symbol Power_Protection:SRV05-4
- removed UR1: 1M, Resistor_SMD:R_0805_2012Metric, symbol device:R
- removed UR2, UR3: 5.1k, Resistor_SMD:R_0805_2012Metric, symbol device:R
- removed USB1: HRO-TYPE-C-31-M-12, Type-C:HRO-TYPE-C-31-M-12-HandSoldering, symbol Type-C:HRO-TYPE-C-31-M-12
- added J1: (no value), symbol Connector:Conn_01x04_Female
Connections:
- net +5V: now also J1.1 (Pin_1)
- net COL0: now also U2.30 (PB6)
- net COL1: now also U2.31 (PC6)
- net COL2: now also U2.32 (PC7)
- net COL3: now also U2.38 (PF5)
- net COL4: now also U2.37 (PF6)
- net COL5: now also U2.25 (PD4)
- net COL6: now also U2.26 (PD6)
- net COL7: now also U2.27 (PD7)
- net COL8: now also U2.28 (PB4)
- net COL9: now also U2.29 (PB5)
- net D+: now also J1.3 (Pin_3)
- net D-: now also J1.2 (Pin_2)
- net GND: now also J1.4 (Pin_4)
- net ROW0: now also U2.41 (PF0); no longer U2.11 (PB3)
- net ROW1: now also U2.40 (PF1); no longer U2.10 (PB2)
- net ROW2: now also U2.39 (PF4); no longer U2.9 (PB1)
- net ROW3: now also D31.1 (K), U2.36 (PF7); no longer U2.8 (PB0)
- no-connect marks 0 -> 12
Other:
- moved on the sheet: R3
